File: tsdz2.kicad_sch (KiCad schematic)
At the start: 6 parts, among them J27 Conn_01x02, J28 Conn_01x06, U4 BTS4140N

Commit message: Before flip
Parts:
- R?: mouser (none) -> 603-AC1206FR-101KL
- R?: value 190k -> 191k; mouser (none) -> 660-RK73H2BTTD1913F
Changed lines of the file:
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@@
+      (effects (font (size 1.27 1.27)) hide)
+    )
+    (property "mouser2" "" (at 72.39 113.03 0)
+      (effects (font (size 1.27 1.27)) hide)
+    )
+    (property "mouser" " 603-AC1206FR-101KL " (at 72.39 113.03 0)
       (effects (font (size 1.27 1.27)) hide)
     )
@@
     )
     (property "tme" "" (at 166.37 87.63 0)
+      (effects (font (size 1.27 1.27)) hide)
+    )
+    (property "mouser2" "" (at 166.37 87.63 0)
       (effects (font (size 1.27 1.27)) hide)
     )
@@
       (effects (font (size 1.27 1.27)) hide)
     )
+    (property "mouser2" "" (at 111.76 107.95 0)
+      (effects (font (size 1.27 1.27)) hide)
+    )
     (pin "4")
     (pin "1")
@@
     )
     (property "tme" "" (at 99.06 85.09 0)
+      (effects (font (size 1.27 1.27)) hide)
+    )
+    (property "mouser2" "" (at 99.06 85.09 0)
       (effects (font (size 1.27 1.27)) hide)
     )
@@
     )
     (property "tme" "" (at 86.36 113.03 0)
+      (effects (font (size 1.27 1.27)) hide)
+    )
+    (property "mouser2" "" (at 86.36 113.03 0)
       (effects (font (size 1.27 1.27)) hide)
     )
@@
       (effects (font (size 1.27 1.27)) (justify left))
     )
-    (property "Value" "190k" (at 81.28 118.11 0)
+    (property "Value" "191k" (at 81.28 118.11 0)
       (effects (font (size 1.27 1.27)) (justify left))
     )
@@
       (effects (font (size 1.27 1.27)) hide)
     )
+    (property "mouser2" "" (at 78.74 116.84 0)
+      (effects (font (size 1.27 1.27)) hide)
+    )
+    (property "mouser" " 660-RK73H2BTTD1913F " (at 78.74 116.84 0)
+      (effects (font (size 1.27 1.27)) hide)
+    )
