File: analog.kicad_sch (KiCad schematic)
At the start: 14 parts, among them J23 Conn_01x04, U5 CD74HC4067M

Commit message: Before flip
Parts:
- removed R?: 4k7, Resistor_SMD:R_1206_3216Metric, symbol Device:R
- R? (x5): value 4k7 -> 10k; mouser (none) -> 603-AC1206FR-0710KL
- R?: value 190k -> 191k; mouser (none) -> 660-RK73H2BTTD1913F
Connections:
- net GND: now also R?.2
Changed lines of the file:
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@@
+      (effects (font (size 1.27 1.27)) hide)
+    )
+    (property "mouser2" "" (at 80.01 88.9 0)
       (effects (font (size 1.27 1.27)) hide)
     )
@@
         (path "/33f5bcad-68ad-4ea6-9034-cdbd4086270c/11d47836-729f-4edd-94b6-45d59ff26291"
           (reference "#PWR053") (unit 1)
-        )
-      )
-    )
-  )
-  (symbol (lib_id "Device:R") (at 111.76 57.15 0) (unit 1)
-    (in_bom yes) (on_board yes) (dnp no)
-    (property "Reference" "R?" (at 114.3 55.8799 0)
-      (effects (font (size 1.27 1.27)) (justify left))
-    )
-    (property "Value" "4k7" (at 114.3 58.4199 0)
-      (effects (font (size 1.27 1.27)) (justify left))
-    )
-    (property "Footprint" "Resistor_SMD:R_1206_3216Metric" (at 109.982 57.15 90)
-      (effects (font (size 1.27 1.27)) hide)
-    )
-    (property "Datasheet" "~" (at 111.76 57.15 0)
-      (effects (font (size 1.27 1.27)) hide)
-    )
-    (property "tme" "" (at 111.76 57.15 0)
-      (effects (font (size 1.27 1.27)) hide)
-    )
-    (pin "1")
-    (pin "2")
-    (instances
-      (project "speedomobile"
-        (path "/33f5bcad-68ad-4ea6-9034-cdbd4086270c"
-          (reference "R?") (unit 1)
-        )
-        (path "/33f5bcad-68ad-4ea6-9034-cdbd4086270c/11d47836-729f-4edd-94b6-45d59ff26291"
-          (reference "R9") (unit 1)
         )
       )
@@
       (effects (font (size 1.27 1.27)) (justify left))
     )
-    (property "Value" "4k7" (at 114.3 50.7999 0)
+    (property "Value" "10k" (at 114.3 50.7999 0)
       (effects (font (size 1.27 1.27)) (justify left))
     )
@@
       (effects (font (size 1.27 1.27)) hide)
     )
+    (property "mouser2" "" (at 111.76 49.53 0)
+      (effects (font (size 1.27 1.27)) hide)
+    )
+    (property "mouser" " 603-AC1206FR-0710KL " (at 111.76 49.53 0)
+      (effects (font (size 1.27 1.27)) hide)
+    )
     (pin "1")
     (pin "2")
@@
     )
     (property "tme" "" (at 157.48 59.69 0)
+      (effects (font (size 1.27 1.27)) hide)
+    )
+    (property "mouser2" "" (at 157.48 59.69 0)
       (effects (font (size 1.27 1.27)) hide)
     )
@@
     )
     (property "tme" "" (at 58.42 120.65 0)
+      (effects (font (size 1.27 1.27)) hide)
+    )
+    (property "mouser2" "" (at 58.42 120.65 0)
       (effects (font (size 1.27 1.27)) hide)
     )
@@
       (effects (font (size 1.27 1.27)) hide)
     )
+    (property "mouser2" "" (at 157.48 39.37 0)
+      (effects (font (size 1.27 1.27)) hide)
+    )
     (pin "3")
     (pin "4")
@@
     )
   )
-  (symbol (lib_id "power:GND") (at 111.76 60.96 0) (unit 1)
-    (in_bom yes) (on_board yes) (dnp no) (fields_autoplaced)
-    (property "Reference" "#PWR056" (at 111.76 67.31 0)
-      (effects (font (size 1.27 1.27)) hide)
-    )
-    (property "Value" "GND" (at 111.76 66.04 0)
-      (effects (font (size 1.27 1.27)))
-    )
-    (property "Footprint" "" (at 111.76 60.96 0)
-      (effects (font (size 1.27 1.27)) hide)
-    )
-    (property "Datasheet" "" (at 111.76 60.96 0)
+  (symbol (lib_id "power:GND") (at 111.76 53.34 0) (unit 1)
+    (in_bom yes) (on_board yes) (dnp no) (fields_autoplaced)
+    (property "Reference" "#PWR056" (at 111.76 59.69 0)
+      (effects (font (size 1.27 1.27)) hide)
+    )
+    (property "Value" "GND" (at 111.76 58.42 0)
+      (effects (font (size 1.27 1.27)))
+    )
+    (property "Footprint" "" (at 111.76 53.34 0)
+      (effects (font (size 1.27 1.27)) hide)
+    )
+    (property "Datasheet" "" (at 111.76 53.34 0)
       (effects (font (size 1.27 1.27)) hide)
     )
@@
       (effects (font (size 1.27 1.27)) (justify left))
     )
-    (property "Value" "4k7" (at 140.97 138.43 0)
+    (property "Value" "10k" (at 140.97 138.43 0)
       (effects (font (size 1.27 1.27)) (justify left))
     )
@@
       (effects (font (size 1.27 1.27)) hide)
     )
+    (property "mouser2" "" (at 138.43 137.16 0)
+      (effects (font (size 1.27 1.27)) hide)
+    )
+    (property "mouser" " 603-AC1206FR-0710KL " (at 138.43 137.16 0)
+      (effects (font (size 1.27 1.27)) hide)
+    )
     (pin "1")
     (pin "2")
@@
     )
     (property "tme" "" (at 104.14 137.16 0)
+      (effects (font (size 1.27 1.27)) hide)
+    )
+    (property "mouser2" "" (at 104.14 137.16 0)
       (effects (font (size 1.27 1.27)) hide)
     )
@@
       (effects (font (size 1.27 1.27)) (justify left))
     )
-    (property "Value" "190k" (at 113.665 43.1799 0)
+    (property "Value" "191k" (at 113.665 43.1799 0)
       (effects (font (size 1.27 1.27)) (justify left))
     )
@@
       (effects (font (size 1.27 1.27)) hide)
     )
+    (property "mouser2" "" (at 111.76 41.91 0)
+      (effects (font (size 1.27 1.27)) hide)
+    )
+    (property "mouser" " 660-RK73H2BTTD1913F " (at 111.76 41.91 0)
+      (effects (font (size 1.27 1.27)) hide)
+    )
     (pin "1")
     (pin "2")
@@
       (effects (font (size 1.27 1.27)) hide)
     )
+    (property "mouser2" "" (at 157.48 78.74 0)
+      (effects (font (size 1.27 1.27)) hide)
+    )
     (pin "2")
     (pin "1")
@@
       (effects (font (size 1.27 1.27)) (justify left))
     )
-    (property "Value" "4k7" (at 154.94 138.43 0)
+    (property "Value" "10k" (at 154.94 138.43 0)
       (effects (font (size 1.27 1.27)) (justify left))
     )
@@
       (effects (font (size 1.27 1.27)) hide)
     )
+    (property "mouser2" "" (at 152.4 137.16 0)
+      (effects (font (size 1.27 1.27)) hide)
+    )
+    (property "mouser" " 603-AC1206FR-0710KL " (at 152.4 137.16 0)
+      (effects (font (size 1.27 1.27)) hide)
+    )
     (pin "1")
     (pin "2")
@@
       (effects (font (size 1.27 1.27)) (justify left))
     )
-    (property "Value" "4k7" (at 154.94 146.05 0)
+    (property "Value" "10k" (at 154.94 146.05 0)
       (effects (font (size 1.27 1.27)) (justify left))
     )
@@
       (effects (font (size 1.27 1.27)) hide)
     )
+    (property "mouser2" "" (at 152.4 144.78 0)
+      (effects (font (size 1.27 1.27)) hide)
+    )
+    (property "mouser" " 603-AC1206FR-0710KL " (at 152.4 144.78 0)
+      (effects (font (size 1.27 1.27)) hide)
+    )
     (pin "1")
     (pin "2")
@@
       (effects (font (size 1.27 1.27)) hide)
     )
+    (property "mouser2" "" (at 157.48 99.06 0)
+      (effects (font (size 1.27 1.27)) hide)
+    )
     (pin "1")
     (pin "2")
@@
       (effects (font (size 1.27 1.27)) (justify left))
     )
-    (property "Value" "4k7" (at 140.97 146.05 0)
+    (property "Value" "10k" (at 140.97 146.05 0)
       (effects (font (size 1.27 1.27)) (justify left))
     )
@@
       (effects (font (size 1.27 1.27)) hide)
     )
+    (property "mouser2" "" (at 138.43 144.78 0)
+      (effects (font (size 1.27 1.27)) hide)
+    )
+    (property "mouser" " 603-AC1206FR-0710KL " (at 138.43 144.78 0)
+      (effects (font (size 1.27 1.27)) hide)
+    )

Commit message: before expansion
Connections:
- net ADC0: now also U5.4 (I5); no longer U5.21 (I10)
- net ADC1: now also U5.5 (I4); no longer U5.20 (I11)
- net ADC2: now also U5.6 (I3); no longer U5.19 (I12)
- net ADC3: now also U5.7 (I2); no longer U5.18 (I13)
- net ADC4: now also U5.8 (I1); no longer U5.17 (I14)
- net AMBIANT: now also U5.17 (I14); no longer U5.7 (I2)
- net BRAKE1: now also U5.19 (I12); no longer U5.5 (I4)
- net BRAKE2: now also U5.20 (I11); no longer U5.4 (I5)
- net I5V: now also U5.16 (I15); no longer U5.9 (I0)
- net Imotor: now also U5.18 (I13); no longer U5.8 (I1)
- net U3V3: now also U5.21 (I10); no longer U5.23 (I8)
- net U5V: now also U5.23 (I8); no longer U5.6 (I3)
- no-connect marks 1 -> 0
Changed lines of the file:
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@@
   (junction (at 152.4 140.97) (diameter 0) (color 0 0 0 0)
   )
-  (no_connect (at 71.12 140.97))
-  (wire (pts (xy 71.12 138.43) (xy 85.09 138.43))
+  (wire (pts (xy 71.12 105.41) (xy 85.09 105.41))
     (stroke (width 0) (type default))
   )
-  (wire (pts (xy 71.12 133.35) (xy 85.09 133.35))
+  (wire (pts (xy 71.12 110.49) (xy 85.09 110.49))
     (stroke (width 0) (type default))
   )
-  (wire (pts (xy 71.12 130.81) (xy 85.09 130.81))
+  (wire (pts (xy 71.12 113.03) (xy 85.09 113.03))
     (stroke (width 0) (type default))
   )
@@
     (stroke (width 0) (type default))
   )
-  (wire (pts (xy 71.12 115.57) (xy 85.09 115.57))
+  (wire (pts (xy 71.12 130.81) (xy 85.09 130.81))
     (stroke (width 0) (type default))
   )
@@
     (stroke (width 0) (type default))
   )
-  (wire (pts (xy 71.12 128.27) (xy 85.09 128.27))
+  (wire (pts (xy 71.12 115.57) (xy 85.09 115.57))
     (stroke (width 0) (type default))
   )
@@
     (stroke (width 0) (type default))
   )
-  (wire (pts (xy 85.09 107.95) (xy 71.12 107.95))
-    (stroke (width 0) (type default))
-  )
-  (wire (pts (xy 71.12 123.19) (xy 85.09 123.19))
+  (wire (pts (xy 85.09 138.43) (xy 71.12 138.43))
     (stroke (width 0) (type default))
   )
   (wire (pts (xy 71.12 120.65) (xy 85.09 120.65))
+    (stroke (width 0) (type default))
+  )
+  (wire (pts (xy 71.12 118.11) (xy 85.09 118.11))
     (stroke (width 0) (type default))
   )
@@
     (stroke (width 0) (type default))
   )
-  (wire (pts (xy 71.12 135.89) (xy 85.09 135.89))
+  (wire (pts (xy 71.12 107.95) (xy 85.09 107.95))
     (stroke (width 0) (type default))
   )
@@
     (stroke (width 0) (type default))
   )
-  (wire (pts (xy 71.12 118.11) (xy 85.09 118.11))
+  (wire (pts (xy 71.12 123.19) (xy 85.09 123.19))
     (stroke (width 0) (type default))
   )
@@
     (stroke (width 0) (type default))
   )
-  (wire (pts (xy 71.12 113.03) (xy 85.09 113.03))
+  (wire (pts (xy 71.12 133.35) (xy 85.09 133.35))
     (stroke (width 0) (type default))
   )
-  (wire (pts (xy 85.09 110.49) (xy 71.12 110.49))
+  (wire (pts (xy 85.09 128.27) (xy 71.12 128.27))
     (stroke (width 0) (type default))
   )
@@
     (effects (font (size 1.27 1.27)) (justify right bottom))
   )
-  (label "U5V" (at 85.09 110.49 180) (fields_autoplaced)
+  (label "U5V" (at 85.09 123.19 180) (fields_autoplaced)
     (effects (font (size 1.27 1.27)) (justify right bottom))
   )
-  (label "AMBIANT" (at 85.09 107.95 180) (fields_autoplaced)
+  (label "AMBIANT" (at 85.09 138.43 180) (fields_autoplaced)
     (effects (font (size 1.27 1.27)) (justify right bottom))
   )
@@
     (effects (font (size 1.27 1.27)) (justify right bottom))
   )
-  (label "BRAKE2" (at 85.09 115.57 180) (fields_autoplaced)
+  (label "BRAKE2" (at 85.09 130.81 180) (fields_autoplaced)
     (effects (font (size 1.27 1.27)) (justify right bottom))
   )
@@
     (effects (font (size 1.27 1.27)) (justify right bottom))
   )
-  (label "U3V3" (at 85.09 123.19 180) (fields_autoplaced)
+  (label "U3V3" (at 85.09 128.27 180) (fields_autoplaced)
     (effects (font (size 1.27 1.27)) (justify right bottom))
   )
-  (label "ADC0" (at 85.09 128.27 180) (fields_autoplaced)
+  (label "ADC0" (at 85.09 115.57 180) (fields_autoplaced)
     (effects (font (size 1.27 1.27)) (justify right bottom))
   )
@@
     (effects (font (size 1.27 1.27)) (justify right bottom))
   )
-  (label "ADC2" (at 85.09 133.35 180) (fields_autoplaced)
+  (label "ADC2" (at 85.09 110.49 180) (fields_autoplaced)
     (effects (font (size 1.27 1.27)) (justify right bottom))
   )
-  (label "BRAKE1" (at 85.09 113.03 180) (fields_autoplaced)
+  (label "BRAKE1" (at 85.09 133.35 180) (fields_autoplaced)
     (effects (font (size 1.27 1.27)) (justify right bottom))
   )
@@
     (effects (font (size 1.27 1.27)) (justify right bottom))
   )
-  (label "ADC4" (at 85.09 138.43 180) (fields_autoplaced)
+  (label "ADC4" (at 85.09 105.41 180) (fields_autoplaced)
     (effects (font (size 1.27 1.27)) (justify right bottom))
   )
-  (label "ADC1" (at 85.09 130.81 180) (fields_autoplaced)
+  (label "ADC1" (at 85.09 113.03 180) (fields_autoplaced)
     (effects (font (size 1.27 1.27)) (justify right bottom))
   )
@@
     (effects (font (size 1.27 1.27)) (justify right bottom))
   )
-  (label "ADC3" (at 85.09 135.89 180) (fields_autoplaced)
+  (label "ADC3" (at 85.09 107.95 180) (fields_autoplaced)
     (effects (font (size 1.27 1.27)) (justify right bottom))
   )
@@
     (effects (font (size 1.27 1.27)) (justify right))
   )
-  (hierarchical_label "Imotor" (shape input) (at 71.12 105.41 0) (fields_autoplaced)
+  (hierarchical_label "Imotor" (shape input) (at 71.12 135.89 0) (fields_autoplaced)
     (effects (font (size 1.27 1.27)) (justify left))
   )
@@
     (effects (font (size 1.27 1.27)) (justify right))
   )
-  (hierarchical_label "I5V" (shape input) (at 71.12 102.87 0) (fields_autoplaced)
+  (hierarchical_label "I5V" (shape input) (at 71.12 140.97 0) (fields_autoplaced)
     (effects (font (size 1.27 1.27)) (justify left))
   )

Commit message: Prepare for merging
Parts:
- added J10: Conn_01x05, Connector_JST:JST_XH_B5B-XH-A_1x05_P2.50mm_Vertical, symbol Connector_Generic:Conn_01x05
- J23: value Conn_01x04 -> XHB4B
- J? (x3): value Conn_01x03 -> XHB3B
Connections:
- net +3V3: now also J10.1 (Pin_1)
- net ADC_SPEED1: now also U5.3 (I6); no longer U5.2 (I7)
- net ADC_SPEED2: now also U5.2 (I7); no longer U5.3 (I6)
- net GND: now also J10.5 (Pin_5)
- net I5V: now also J10.4 (Pin_4)
- net Imotor: now also J10.3 (Pin_3)
- net U5V: now also U5.22 (I9); no longer U5.23 (I8)
- net VBATADC: now also U5.9 (I0); no longer U5.22 (I9)
- new net Iaux: J10.2 (Pin_2), U5.23 (I8)
