File: i2c.kicad_sch (KiCad schematic)
At the start: 36 parts, among them J1 Conn_01x04, J2 Conn_01x04, J3 Conn_01x04, J37 Conn_01x02, J38 Conn_01x03, J4 Conn_01x04, J5 Conn_01x04, J8 Conn_01x04, J9 Conn_Coaxial, Q5 BSS138, Q6 BSS138, U10 NEO-M9N, U11 PCF8574, U12 PCF8574

Commit message: JLCJLCJLCJLC
Parts:
- removed J5, J?: Conn_01x04, Connector_JST:JST_XH_B4B-XH-A_1x04_P2.50mm_Vertical, symbol Connector_Generic:Conn_01x04
- removed Q5, Q6: BSS138, Package_TO_SOT_SMD:SOT-23, symbol Transistor_FET:BSS138
- removed R21, R22: 4k7, Resistor_SMD:R_1206_3216Metric, symbol Device:R
- added J5: Conn_01x05, Connector_JST:JST_XH_B5B-XH-A_1x05_P2.50mm_Vertical, symbol Connector_Generic:Conn_01x05
- added J6: Conn_01x04, Connector_JST:JST_XH_B4B-XH-A_1x04_P2.50mm_Vertical, symbol Connector_Generic:Conn_01x04
Connections:
- net +3V3: now also J5.2 (Pin_2), J6.1 (Pin_1)
- net +5VL: now also J5.1 (Pin_1)
- net GND: now also J5.5 (Pin_5), J6.4 (Pin_4)
- net SCL: now also J5.4 (Pin_4), J6.3 (Pin_3)
- net SDA: now also J5.3 (Pin_3), J6.2 (Pin_2)
Other:
- note removed: "MFRC522 0x06"

Commit message: Before flip
Parts:
- C20: footprint Capacitor_SMD:C_1206_3216Metric -> Capacitor_SMD:C_0603_1608Metric; mouser 80-C1206C104K5R -> 187-CL10B104KA8NNWC
- L1: footprint Inductor_SMD:L_1206_3216Metric -> Inductor_SMD:L_0603_1608Metric; mouser (none) -> 871-B82496C3270J
- R18: footprint Resistor_SMD:R_1206_3216Metric -> Resistor_SMD:R_0603_1608Metric; mouser (none) -> 660-SG73P1JTTD20R0F
- R19, R20, R27, R28: mouser (none) -> 791-WR12X4701FTL
- R23, R24: value 2k -> 1k; mouser (none) -> 603-AC1206FR-101KL
- R25, R26: mouser (none) -> 603-AC1206FR-101KL
Connections:
- net PPS: now reaches U10.3 (TIMEPULSE)
- no-connect marks 15 -> 14
Changed lines of the file:
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@@
   (no_connect (at 217.17 139.7))
   (no_connect (at 90.17 153.67))
-  (no_connect (at 125.73 153.67))
   (no_connect (at 125.73 140.97))
   (no_connect (at 90.17 133.35))
@@
     (effects (font (size 1.27 1.27)) (justify left))
   )
+  (hierarchical_label "PPS" (shape output) (at 125.73 153.67 0) (fields_autoplaced)
+    (effects (font (size 1.27 1.27)) (justify left))
+  )
   (symbol (lib_id "power:GND") (at 249.555 80.645 0) (unit 1)
     (in_bom yes) (on_board yes) (dnp no) (fields_autoplaced)
@@
       (effects (font (size 1.27 1.27)) (justify left))
     )
-    (property "Value" "2k" (at 231.14 27.94 0)
+    (property "Value" "1k" (at 231.14 27.94 0)
       (effects (font (size 1.27 1.27)) (justify left))
     )
@@
       (effects (font (size 1.27 1.27)) hide)
     )
+    (property "mouser2" "" (at 228.6 26.67 0)
+      (effects (font (size 1.27 1.27)) hide)
+    )
+    (property "mouser" " 603-AC1206FR-101KL " (at 228.6 26.67 0)
+      (effects (font (size 1.27 1.27)) hide)
+    )
     (pin "2")
     (pin "1")
@@
       (effects (font (size 1.27 1.27)))
     )
-    (property "Footprint" "Capacitor_SMD:C_1206_3216Metric" (at 152.4 134.9248 0)
+    (property "Footprint" "Capacitor_SMD:C_0603_1608Metric" (at 152.4 134.9248 0)
       (effects (font (size 1.27 1.27)) hide)
     )
@@
       (effects (font (size 1.27 1.27)) hide)
     )
-    (property "mouser" " 80-C1206C104K5R " (at 148.59 135.89 0)
+    (property "mouser" " 187-CL10B104KA8NNWC " (at 148.59 135.89 0)
       (effects (font (size 1.27 1.27)) hide)
     )
@@
       (effects (font (size 1.27 1.27)) hide)
     )
+    (property "mouser2" "" (at 148.59 135.89 0)
+      (effects (font (size 1.27 1.27)) hide)
+    )
     (pin "2")
     (pin "1")
@@
       (effects (font (size 1.27 1.27)) hide)
     )
+    (property "mouser2" "" (at 193.04 26.67 0)
+      (effects (font (size 1.27 1.27)) hide)
+    )
+    (property "mouser" " 791-WR12X4701FTL " (at 193.04 26.67 0)
+      (effects (font (size 1.27 1.27)) hide)
+    )
     (pin "2")
     (pin "1")
@@
     )
     (property "tme" "" (at 30.48 135.89 0)
+      (effects (font (size 1.27 1.27)) hide)
+    )
+    (property "mouser2" "" (at 30.48 135.89 0)
       (effects (font (size 1.27 1.27)) hide)
     )
@@
       (effects (font (size 1.27 1.27)) hide)
     )
+    (property "mouser2" "" (at 246.38 146.05 0)
+      (effects (font (size 1.27 1.27)) hide)
+    )
     (pin "2")
     (pin "1")
@@
       (effects (font (size 1.27 1.27)) hide)
     )
+    (property "mouser2" "" (at 105.41 111.76 0)
+      (effects (font (size 1.27 1.27)) hide)
+    )
     (pin "3")
     (pin "2")
@@
     )
     (property "tme" "" (at 80.01 115.57 0)
+      (effects (font (size 1.27 1.27)) hide)
+    )
+    (property "mouser2" "" (at 80.01 115.57 0)
       (effects (font (size 1.27 1.27)) hide)
     )
@@
       (effects (font (size 1.27 1.27)) hide)
     )
+    (property "mouser2" "" (at 254 156.21 0)
+      (effects (font (size 1.27 1.27)) hide)
+    )
+    (property "mouser" " 603-AC1206FR-101KL " (at 254 156.21 0)
+      (effects (font (size 1.27 1.27)) hide)
+    )
     (pin "1")
     (pin "2")
@@
     )
     (property "tme" "" (at 175.26 92.71 0)
+      (effects (font (size 1.27 1.27)) hide)
+    )
+    (property "mouser2" "" (at 175.26 92.71 0)
       (effects (font (size 1.27 1.27)) hide)
     )
@@
       (effects (font (size 1.27 1.27)) hide)
     )
+    (property "mouser2" "" (at 60.96 140.97 0)
+      (effects (font (size 1.27 1.27)) hide)
+    )
     (pin "3")
     (pin "2")
@@
       (effects (font (size 1.27 1.27)) (justify left))
     )
-    (property "Footprint" "Resistor_SMD:R_1206_3216Metric" (at 135.382 132.08 90)
+    (property "Footprint" "Resistor_SMD:R_0603_1608Metric" (at 135.382 132.08 90)
       (effects (font (size 1.27 1.27)) hide)
     )
@@
       (effects (font (size 1.27 1.27)) hide)
     )
+    (property "mouser2" "" (at 137.16 132.08 0)
+      (effects (font (size 1.27 1.27)) hide)
+    )
+    (property "mouser" " 660-SG73P1JTTD20R0F " (at 137.16 132.08 0)
+      (effects (font (size 1.27 1.27)) hide)
+    )
     (pin "1")
     (pin "2")
@@
       (effects (font (size 1.27 1.27)) hide)
     )
+    (property "mouser2" "" (at 201.93 26.67 0)
+      (effects (font (size 1.27 1.27)) hide)
+    )
+    (property "mouser" " 791-WR12X4701FTL " (at 201.93 26.67 0)
+      (effects (font (size 1.27 1.27)) hide)
+    )
     (pin "2")
     (pin "1")
@@
     )
     (property "tme" "" (at 204.47 137.16 0)
+      (effects (font (size 1.27 1.27)) hide)
+    )
+    (property "mouser2" "" (at 204.47 137.16 0)
       (effects (font (size 1.27 1.27)) hide)
     )
@@
       (effects (font (size 1.27 1.27)) hide)
     )
+    (property "mouser2" "" (at 261.62 113.03 0)
+      (effects (font (size 1.27 1.27)) hide)
+    )
     (pin "2")
     (pin "1")
@@
     )
     (property "tme" "" (at 107.95 146.05 0)
+      (effects (font (size 1.27 1.27)) hide)
+    )
+    (property "mouser2" "" (at 107.95 146.05 0)
       (effects (font (size 1.27 1.27)) hide)
     )
@@
       (effects (font (size 1.27 1.27)) hide)
     )
+    (property "mouser2" "" (at 137.16 149.86 0)
+      (effects (font (size 1.27 1.27)) hide)
+    )
     (pin "2")
     (pin "1")
@@
     )
     (property "tme" "" (at 30.48 69.85 0)
+      (effects (font (size 1.27 1.27)) hide)
+    )
+    (property "mouser2" "" (at 30.48 69.85 0)
       (effects (font (size 1.27 1.27)) hide)
     )
@@
       (effects (font (size 1.27 1.27)) hide)
     )
+    (property "mouser2" "" (at 30.48 91.44 0)
+      (effects (font (size 1.27 1.27)) hide)
+    )
     (pin "4")
     (pin "3")
@@
       (effects (font (size 1.27 1.27)) hide)
     )
+    (property "mouser2" "" (at 254 146.05 0)
+      (effects (font (size 1.27 1.27)) hide)
+    )
+    (property "mouser" " 603-AC1206FR-101KL " (at 254 146.05 0)
+      (effects (font (size 1.27 1.27)) hide)
+    )
     (pin "1")
     (pin "2")
@@
     )
     (property "tme" "" (at 181.61 154.94 0)
+      (effects (font (size 1.27 1.27)) hide)
+    )
+    (property "mouser2" "" (at 181.61 154.94 0)
       (effects (font (size 1.27 1.27)) hide)
     )
@@
       (effects (font (size 1.27 1.27)) hide)
     )
+    (property "mouser2" "" (at 74.93 66.04 0)
+      (effects (font (size 1.27 1.27)) hide)
+    )
     (pin "4")
     (pin "3")
@@
       (effects (font (size 1.27 1.27)) hide)
     )
+    (property "mouser2" "" (at 30.48 114.3 0)
+      (effects (font (size 1.27 1.27)) hide)
+    )
     (pin "4")
     (pin "3")
@@
       (effects (font (size 1.27 1.27)) hide)
     )
+    (property "mouser2" "" (at 246.38 156.21 0)
+      (effects (font (size 1.27 1.27)) hide)
+    )
     (pin "2")
     (pin "1")
@@
       (effects (font (size 1.27 1.27)) hide)
     )
+    (property "mouser2" "" (at 245.745 76.835 0)
+      (effects (font (size 1.27 1.27)) hide)
+    )
+    (property "mouser" " 791-WR12X4701FTL " (at 245.745 76.835 0)
+      (effects (font (size 1.27 1.27)) hide)
+    )
     (pin "1")
     (pin "2")
@@
       (effects (font (size 1.27 1.27)) hide)
     )
+    (property "mouser2" "" (at 254 76.835 0)
+      (effects (font (size 1.27 1.27)) hide)
+    )
+    (property "mouser" " 791-WR12X4701FTL " (at 254 76.835 0)
+      (effects (font (size 1.27 1.27)) hide)
+    )
     (pin "1")
     (pin "2")
@@
       (effects (font (size 1.27 1.27)) (justify left))
     )
-    (property "Value" "2k" (at 240.03 27.94 0)
+    (property "Value" "1k" (at 240.03 27.94 0)
       (effects (font (size 1.27 1.27)) (justify left))
     )
@@
       (effects (font (size 1.27 1.27)) hide)
     )
+    (property "mouser2" "" (at 237.49 26.67 0)
+      (effects (font (size 1.27 1.27)) hide)
+    )
+    (property "mouser" " 603-AC1206FR-101KL " (at 237.49 26.67 0)
+      (effects (font (size 1.27 1.27)) hide)
+    )
     (pin "2")
     (pin "1")
@@
     )
     (property "tme" "" (at 185.42 63.5 0)
+      (effects (font (size 1.27 1.27)) hide)
+    )
+    (property "mouser2" "" (at 185.42 63.5 0)
       (effects (font (size 1.27 1.27)) hide)
     )
@@
     )
     (property "tme" "" (at 235.585 90.17 0)
+      (effects (font (size 1.27 1.27)) hide)
+    )
+    (property "mouser2" "" (at 235.585 90.17 0)
       (effects (font (size 1.27 1.27)) hide)
     )
@@
       (effects (font (size 1.27 1.27)) hide)
     )
+    (property "mouser2" "" (at 74.93 90.17 0)
+      (effects (font (size 1.27 1.27)) hide)
+    )
     (pin "1")
     (pin "2")
@@
       (effects (font (size 1.27 1.27)) (justify left))
     )
-    (property "Footprint" "Inductor_SMD:L_1206_3216Metric" (at 137.16 142.24 0)
+    (property "Footprint" "Inductor_SMD:L_0603_1608Metric" (at 137.16 142.24 0)
       (effects (font (size 1.27 1.27)) hide)
     )
@@
       (effects (font (size 1.27 1.27)) hide)
     )
+    (property "mouser2" "" (at 137.16 142.24 0)
+      (effects (font (size 1.27 1.27)) hide)
+    )
+    (property "mouser" " 871-B82496C3270J " (at 137.16 142.24 0)
+      (effects (font (size 1.27 1.27)) hide)
+    )
     (pin "2")
     (pin "1")
@@
       (effects (font (size 1.27 1.27)) hide)
     )
+    (property "mouser2" "" (at 151.13 146.05 0)
+      (effects (font (size 1.27 1.27)) hide)
+    )
     (pin "1")
     (pin "2")
@@
       (effects (font (size 1.27 1.27)) hide)
     )
+    (property "mouser2" "" (at 95.25 40.64 0)
+      (effects (font (size 1.27 1.27)) hide)
+    )

Commit message: before expansion
Parts:
- removed J38: Conn_01x03, Connector_PinHeader_2.54mm:PinHeader_1x03_P2.54mm_Vertical, symbol Connector_Generic:Conn_01x03
- removed J8: Conn_01x04, Connector_PinHeader_2.54mm:PinHeader_1x04_P2.54mm_Vertical, symbol Connector_Generic:Conn_01x04
- added J38: Conn_01x04, Connector_JST:JST_XH_B4B-XH-A_1x04_P2.50mm_Vertical, symbol Connector_Generic:Conn_01x04
- added J8: Conn_01x03, Connector_PinHeader_2.54mm:PinHeader_1x03_P2.54mm_Vertical, symbol Connector_Generic:Conn_01x03
Connections:
- net +3V3: now also U11.1 (A0), J38.2 (Pin_2); no longer U12.1 (A0)
- net +5VL: now also J38.1 (Pin_1)
- net GND: now also U12.1 (A0), J38.4 (Pin_4), J8.3 (Pin_3); no longer U11.1 (A0)
- net at U10.22 (V_BCKP): now also J38.3 (Pin_3)
- net at U10.21 (RXD/SPI_MOSI): now also J8.1 (Pin_1)
- net at U10.20 (TXD/SPI_MISO): now also J8.2 (Pin_2)

Commit message: Prepare for merging
Parts:
- removed C20: 100n, Capacitor_SMD:C_0603_1608Metric, symbol Device:C
- removed C?: 1u, Capacitor_SMD:C_1206_3216Metric, symbol Device:C
- removed D4: 1.5KExxA, Diode_SMD:D_0603_1608Metric, symbol Diode:1.5KExxA
- removed J38: Conn_01x04, Connector_JST:JST_XH_B4B-XH-A_1x04_P2.50mm_Vertical, symbol Connector_Generic:Conn_01x04
- removed J8: Conn_01x03, Connector_PinHeader_2.54mm:PinHeader_1x03_P2.54mm_Vertical, symbol Connector_Generic:Conn_01x03
- removed J9: Conn_Coaxial, Connector_Coaxial:U.FL_Hirose_U.FL-R-SMT-1_Vertical, symbol Connector:Conn_Coaxial
- removed L1: 27nH, Inductor_SMD:L_0603_1608Metric, symbol Device:L
- removed R18: 20, Resistor_SMD:R_0603_1608Metric, symbol Device:R
- removed U10: NEO-M9N, RF_GPS:ublox_NEO, symbol RF_GPS:NEO-M9N
Connections:
- net FAST_SCL: no longer J1.3 (Pin_3), J2.3 (Pin_3)
- net FAST_SDA: no longer J1.2 (Pin_2), J2.2 (Pin_2)
- net GND: no longer U?.6 (CS_AG), U?.7 (CS_M), U?.8 (MISO_AG), U?.9 (MISO_M)
- net HONK: now also U11.12 (P7); no longer U11.11 (P6)
- net RESET_M9N: now also U11.9 (P4); no longer U11.12 (P7)
- net SCL: now also J1.3 (Pin_3), J2.3 (Pin_3)
- net SDA: now also J1.2 (Pin_2), J2.2 (Pin_2)
- net TSDZ2_BRAKE: now also U11.10 (P5); no longer U11.9 (P4)
- net TSDZ2_ON: now also U11.11 (P6); no longer U11.10 (P5)
- no-connect marks 14 -> 13
Other:
- removed sheet led ribbon
- note added: "Acc+Gyr 0x6A Magn 0x1C"
- note removed: "Acc+Gyr 0xD4 Magn 0x38"
- note removed: "GPIO 0x40"
- note removed: "GPIO 0x42"
