File: power.kicad_sch (KiCad schematic)
At the start: 36 parts, among them J20 Conn_01x03, J21 Conn_01x03, J33 Conn_01x03, U8 V48SD

Commit message: JLCJLCJLCJLC
Parts:
- NT3, NT4: footprint NetTie:NetTie-2_SMD_Pad2.0mm -> additional:NetTie-2_SMD_Pad2.0mm-3,6mm
- TH? (x5): footprint Resistor_SMD:R_1812_4532Metric -> Resistor_SMD:R_1210_3225Metric; mouser 603-SMD1812B300TFT -> 504-PTSLR12106V300
Changed lines of the file:
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@@
       (effects (font (size 1.27 1.27)))
     )
-    (property "Footprint" "NetTie:NetTie-2_SMD_Pad2.0mm" (at 88.9 175.895 0)
+    (property "Footprint" "additional:NetTie-2_SMD_Pad2.0mm-3,6mm" (at 88.9 175.895 0)
       (effects (font (size 1.27 1.27)) hide)
     )
@@
       (effects (font (size 1.27 1.27)))
     )
-    (property "Footprint" "NetTie:NetTie-2_SMD_Pad2.0mm" (at 88.9 180.975 0)
+    (property "Footprint" "additional:NetTie-2_SMD_Pad2.0mm-3,6mm" (at 88.9 180.975 0)
       (effects (font (size 1.27 1.27)) hide)
     )
@@
       (effects (font (size 1.27 1.27)))
     )
-    (property "Footprint" "Resistor_SMD:R_1812_4532Metric" (at 147.32 162.56 0)
+    (property "Footprint" "Resistor_SMD:R_1210_3225Metric" (at 147.32 162.56 0)
       (effects (font (size 1.27 1.27)) (justify left) hide)
     )
@@
       (effects (font (size 1.27 1.27)) hide)
     )
-    (property "mouser" " 603-SMD1812B300TFT " (at 142.24 163.83 0)
+    (property "mouser" " 504-PTSLR12106V300" (at 142.24 163.83 0)
       (effects (font (size 1.27 1.27)) hide)
     )
@@
       (effects (font (size 1.27 1.27)))
     )
-    (property "Footprint" "Resistor_SMD:R_1812_4532Metric" (at 226.06 41.91 0)
+    (property "Footprint" "Resistor_SMD:R_1210_3225Metric" (at 226.06 41.91 0)
       (effects (font (size 1.27 1.27)) (justify left) hide)
     )
@@
       (effects (font (size 1.27 1.27)) hide)
     )
-    (property "mouser" " 603-SMD1812B300TFT " (at 220.98 43.18 0)
+    (property "mouser" " 504-PTSLR12106V300" (at 220.98 43.18 0)
       (effects (font (size 1.27 1.27)) hide)
     )
@@
       (effects (font (size 1.27 1.27)))
     )
-    (property "Footprint" "Resistor_SMD:R_1812_4532Metric" (at 147.32 123.19 0)
+    (property "Footprint" "Resistor_SMD:R_1210_3225Metric" (at 147.32 123.19 0)
       (effects (font (size 1.27 1.27)) (justify left) hide)
     )
@@
       (effects (font (size 1.27 1.27)) hide)
     )
-    (property "mouser" " 603-SMD1812B300TFT " (at 142.24 124.46 0)
+    (property "mouser" " 504-PTSLR12106V300" (at 142.24 124.46 0)
       (effects (font (size 1.27 1.27)) hide)
     )
@@
       (effects (font (size 1.27 1.27)))
     )
-    (property "Footprint" "Resistor_SMD:R_1812_4532Metric" (at 147.32 137.16 0)
+    (property "Footprint" "Resistor_SMD:R_1210_3225Metric" (at 147.32 137.16 0)
       (effects (font (size 1.27 1.27)) (justify left) hide)
     )
@@
       (effects (font (size 1.27 1.27)) hide)
     )
-    (property "mouser" " 603-SMD1812B300TFT " (at 142.24 138.43 0)
+    (property "mouser" " 504-PTSLR12106V300" (at 142.24 138.43 0)
       (effects (font (size 1.27 1.27)) hide)
     )
@@
       (effects (font (size 1.27 1.27)))
     )
-    (property "Footprint" "Resistor_SMD:R_1812_4532Metric" (at 147.32 151.13 0)
+    (property "Footprint" "Resistor_SMD:R_1210_3225Metric" (at 147.32 151.13 0)
       (effects (font (size 1.27 1.27)) (justify left) hide)
     )
@@
       (effects (font (size 1.27 1.27)) hide)
     )
-    (property "mouser" " 603-SMD1812B300TFT " (at 142.24 152.4 0)
-      (effects (font (size 1.27 1.27)) hide)
-    )
+    (property "mouser" " 504-PTSLR12106V300" (at 142.24 152.4 0)
+      (effects (font (size 1.27 1.27)) hide)
+    )

Commit message: 2 layers!
Parts:
- removed J20, J21: Conn_01x03, Connector_JST:JST_XH_B3B-XH-A_1x03_P2.50mm_Vertical, symbol Connector_Generic:Conn_01x03
- removed NT1: NetTie_2, NetTie:NetTie-2_SMD_Pad0.5mm, symbol Device:NetTie_2
- removed NT3, NT4: NetTie_2, additional:NetTie-2_SMD_Pad2.0mm-3,6mm, symbol Device:NetTie_2
- removed Q? (x2): DMT6012LSS, Package_SO:SOIC-8_3.9x4.9mm_P1.27mm, symbol Transistor_FET:IRF7403
- removed R? (x2): 1k, Resistor_SMD:R_1206_3216Metric, symbol Device:R
- removed R? (x2): 190k, Resistor_SMD:R_1206_3216Metric, symbol Device:R
- added J? (x2): Conn_01x02, Connector_JST:JST_XH_B2B-XH-A_1x02_P2.50mm_Vertical, symbol Connector_Generic:Conn_01x02
Connections:
- net GNDPWR is gone; now on net GND: J?.2 (Pin_2), J?.2 (Pin_2)
- net +5VL: now also U8.7 (Sense+)
- net GND: now also J?.2 (Pin_2), J?.2 (Pin_2)
- net PWR1: now also J?.1 (Pin_1)
- net PWR2: now also J?.1 (Pin_1)

Commit message: before expansion
Parts:
- removed C12: 100u, Capacitor_THT:CP_Radial_D6.3mm_P2.50mm, symbol Device:C_Polarized
- added C12: 22u, Capacitor_SMD:C_1210_3225Metric, symbol Device:C
Connections:
- net +5VL: now also C12.1
- net GND: now also C12.2
Changed lines of the file:
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@@
+    )
+  )
+  (symbol (lib_id "Device:C") (at 234.95 69.85 0) (unit 1)
+    (in_bom yes) (on_board yes) (dnp no) (fields_autoplaced)
+    (property "Reference" "C12" (at 238.76 68.58 0)
+      (effects (font (size 1.27 1.27)) (justify left))
+    )
+    (property "Value" "22u" (at 238.76 71.12 0)
+      (effects (font (size 1.27 1.27)) (justify left))
+    )
+    (property "Footprint" "Capacitor_SMD:C_1210_3225Metric" (at 235.9152 73.66 0)
+      (effects (font (size 1.27 1.27)) hide)
+    )
+    (property "Datasheet" "~" (at 234.95 69.85 0)
+      (effects (font (size 1.27 1.27)) hide)
+    )
+    (property "Mouser" "CL32B226MOJNNNE" (at 234.95 69.85 0)
+      (effects (font (size 1.27 1.27)) hide)
+    )
+    (property "mouser" "CL32B226MOJNNNE" (at 234.95 69.85 0)
+      (effects (font (size 1.27 1.27)) hide)
+    )
+    (property "tme" "" (at 234.95 69.85 0)
+      (effects (font (size 1.27 1.27)) hide)
+    )
+    (property "mouser2" "" (at 234.95 69.85 0)
+      (effects (font (size 1.27 1.27)) hide)
+    )
+    (pin "2")
+    (pin "1")
+    (instances
+      (project "speedomobile"
+        (path "/33f5bcad-68ad-4ea6-9034-cdbd4086270c/f11e76c2-c975-435e-b3f1-8c0be3fa1a36"
+          (reference "C12") (unit 1)
+        )
+      )
     )
   )
@@
         )
       )
-    )
-  )
-  (symbol (lib_id "Device:C_Polarized") (at 234.95 69.85 0) (unit 1)
-    (in_bom yes) (on_board yes) (dnp no) (fields_autoplaced)
-    (property "Reference" "C12" (at 238.76 67.691 0)
-      (effects (font (size 1.27 1.27)) (justify left))
-    )
-    (property "Value" "100u" (at 238.76 70.231 0)
-      (effects (font (size 1.27 1.27)) (justify left))
-    )
-    (property "Footprint" "Capacitor_THT:CP_Radial_D6.3mm_P2.50mm" (at 235.9152 73.66 0)
-      (effects (font (size 1.27 1.27)) hide)
-    )
-    (property "Datasheet" "~" (at 234.95 69.85 0)
-      (effects (font (size 1.27 1.27)) hide)
-    )
-    (property "Mouser" "A750EK107M1CAAE018" (at 234.95 69.85 0)
-      (effects (font (size 1.27 1.27)) hide)
-    )
-    (property "mouser" "A750EK107M1CAAE018" (at 234.95 69.85 0)
-      (effects (font (size 1.27 1.27)) hide)
-    )
-    (property "tme" "" (at 234.95 69.85 0)
-      (effects (font (size 1.27 1.27)) hide)
-    )
-    (property "mouser2" "" (at 234.95 69.85 0)
-      (effects (font (size 1.27 1.27)) hide)
-    )
-    (pin "2")
-    (pin "1")
-    (instances
-      (project "speedomobile"
-        (path "/33f5bcad-68ad-4ea6-9034-cdbd4086270c/f11e76c2-c975-435e-b3f1-8c0be3fa1a36"
-          (reference "C12") (unit 1)
-        )
-      )

Commit message: Prepare for merging
Parts:
- removed C10, C15, C16: 22u, Capacitor_SMD:C_1210_3225Metric, symbol Device:C
- removed C14: 100u, Capacitor_THT:CP_Radial_D6.3mm_P2.50mm, symbol Device:C_Polarized
- removed C6, C7, C8, C9: 1u, Capacitor_SMD:C_1206_3216Metric, symbol Device:C
- removed J33: Conn_01x03, Connector_PinHeader_2.54mm:PinHeader_1x03_P2.54mm_Vertical, symbol Connector_Generic:Conn_01x03
- removed U? (x2): MCS1802, Package_SO:SOIC-8_3.9x4.9mm_P1.27mm, symbol Sensor_Current:ACS725xLCTR-50AB
- added C10: 220u, Capacitor_THT:CP_Radial_D16.0mm_P7.50mm, symbol Device:C_Polarized
- added J?: Conn_01x02, Connector_AMASS:AMASS_XT60-F_1x02_P7.20mm_Vertical, symbol Connector_Generic:Conn_01x02
- C13: value 22u -> 1u; footprint Capacitor_SMD:C_1210_3225Metric -> Capacitor_SMD:C_1206_3216Metric; Mouser CL32B226MOJNNNE -> (none); mouser CL32B226MOJNNNE -> 187-CL31B105KBHNFNE
- U8: footprint additional:V48D -> additional:VCB48
Connections:
- net +5V: now also C10.1
- net -BATT: now also U8.2 (ON/~{OFF}), J?.1 (Pin_1)
- net GND: now also C10.2
- new net aux48v: J?.2 (Pin_2)
- no-connect marks 2 -> 1
Other:
- added sheet current sensor (current_sensor.kicad_sch)
- added sheet current sensor1 (current_sensor.kicad_sch)
- added sheet current sensor2 (current_sensor.kicad_sch)
- moved on the sheet: C12
