File: rfid.kicad_sch (KiCad schematic)
At the start: 3 parts

Commit message: before expansion
Parts:
- removed C?: 100u, Capacitor_THT:CP_Radial_D6.3mm_P2.50mm, symbol Device:C_Polarized
- added C12: 22u, Capacitor_SMD:C_1210_3225Metric, symbol Device:C
Connections:
- net +3V3: now also C12.1
- net GND: now also C12.2
Changed lines of the file:
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@@
+    )
+  )
+  (symbol (lib_id "Device:C") (at 200.66 101.6 0) (unit 1)
+    (in_bom yes) (on_board yes) (dnp no) (fields_autoplaced)
+    (property "Reference" "C12" (at 204.47 100.33 0)
+      (effects (font (size 1.27 1.27)) (justify left))
+    )
+    (property "Value" "22u" (at 204.47 102.87 0)
+      (effects (font (size 1.27 1.27)) (justify left))
+    )
+    (property "Footprint" "Capacitor_SMD:C_1210_3225Metric" (at 201.6252 105.41 0)
+      (effects (font (size 1.27 1.27)) hide)
+    )
+    (property "Datasheet" "~" (at 200.66 101.6 0)
+      (effects (font (size 1.27 1.27)) hide)
+    )
+    (property "Mouser" "CL32B226MOJNNNE" (at 200.66 101.6 0)
+      (effects (font (size 1.27 1.27)) hide)
+    )
+    (property "mouser" "CL32B226MOJNNNE" (at 200.66 101.6 0)
+      (effects (font (size 1.27 1.27)) hide)
+    )
+    (property "tme" "" (at 200.66 101.6 0)
+      (effects (font (size 1.27 1.27)) hide)
+    )
+    (property "mouser2" "" (at 200.66 101.6 0)
+      (effects (font (size 1.27 1.27)) hide)
+    )
+    (pin "2")
+    (pin "1")
+    (instances
+      (project "speedomobile"
+        (path "/33f5bcad-68ad-4ea6-9034-cdbd4086270c/f11e76c2-c975-435e-b3f1-8c0be3fa1a36"
+          (reference "C12") (unit 1)
+        )
+        (path "/33f5bcad-68ad-4ea6-9034-cdbd4086270c/51c364bc-8dcb-4f10-88b1-180da7ba62ce"
+          (reference "C25") (unit 1)
+        )
+      )
     )
   )
@@
         )
       )
-    )
-  )
-  (symbol (lib_id "Device:C_Polarized") (at 200.66 101.6 0) (unit 1)
-    (in_bom yes) (on_board yes) (dnp no) (fields_autoplaced)
-    (property "Reference" "C?" (at 204.47 99.441 0)
-      (effects (font (size 1.27 1.27)) (justify left))
-    )
-    (property "Value" "100u" (at 204.47 101.981 0)
-      (effects (font (size 1.27 1.27)) (justify left))
-    )
-    (property "Footprint" "Capacitor_THT:CP_Radial_D6.3mm_P2.50mm" (at 201.6252 105.41 0)
-      (effects (font (size 1.27 1.27)) hide)
-    )
-    (property "Datasheet" "~" (at 200.66 101.6 0)
-      (effects (font (size 1.27 1.27)) hide)
-    )
-    (property "Mouser" "A750EK107M1CAAE018" (at 200.66 101.6 0)
-      (effects (font (size 1.27 1.27)) hide)
-    )
-    (property "mouser" "A750EK107M1CAAE018" (at 200.66 101.6 0)
-      (effects (font (size 1.27 1.27)) hide)
-    )
-    (property "tme" "" (at 200.66 101.6 0)
-      (effects (font (size 1.27 1.27)) hide)
-    )
-    (property "mouser2" "" (at 200.66 101.6 0)
-      (effects (font (size 1.27 1.27)) hide)
-    )
-    (pin "2")
-    (pin "1")
-    (instances
-      (project "speedomobile"
-        (path "/33f5bcad-68ad-4ea6-9034-cdbd4086270c/f11e76c2-c975-435e-b3f1-8c0be3fa1a36"
-          (reference "C?") (unit 1)
-        )
-        (path "/33f5bcad-68ad-4ea6-9034-cdbd4086270c/51c364bc-8dcb-4f10-88b1-180da7ba62ce"
-          (reference "C17") (unit 1)
-        )
-      )

Commit message: Prepare for merging
Parts:
- gave numbers to parts that had none: 1
- renumbered C12 to C25
Changed lines of the file:
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@@
   (symbol (lib_id "power:GND") (at 200.66 105.41 0) (unit 1)
     (in_bom yes) (on_board yes) (dnp no) (fields_autoplaced)
-    (property "Reference" "#PWR?" (at 200.66 111.76 0)
+    (property "Reference" "#PWR0114" (at 200.66 111.76 0)
       (effects (font (size 1.27 1.27)) hide)
     )
@@
     (instances
       (project "speedomobile"
-        (path "/33f5bcad-68ad-4ea6-9034-cdbd4086270c/f11e76c2-c975-435e-b3f1-8c0be3fa1a36"
-          (reference "#PWR?") (unit 1)
-        )
         (path "/33f5bcad-68ad-4ea6-9034-cdbd4086270c/51c364bc-8dcb-4f10-88b1-180da7ba62ce"
           (reference "#PWR0114") (unit 1)
@@
   (symbol (lib_id "Device:C") (at 200.66 101.6 0) (unit 1)
     (in_bom yes) (on_board yes) (dnp no) (fields_autoplaced)
-    (property "Reference" "C12" (at 204.47 100.33 0)
+    (property "Reference" "C25" (at 204.47 100.33 0)
       (effects (font (size 1.27 1.27)) (justify left))
     )
@@
     (instances
       (project "speedomobile"
-        (path "/33f5bcad-68ad-4ea6-9034-cdbd4086270c/f11e76c2-c975-435e-b3f1-8c0be3fa1a36"
-          (reference "C12") (unit 1)
-        )
         (path "/33f5bcad-68ad-4ea6-9034-cdbd4086270c/51c364bc-8dcb-4f10-88b1-180da7ba62ce"
           (reference "C25") (unit 1)
@@
   (symbol (lib_id "power:+3V3") (at 200.66 97.79 0) (unit 1)
     (in_bom yes) (on_board yes) (dnp no) (fields_autoplaced)
-    (property "Reference" "#PWR?" (at 200.66 101.6 0)
+    (property "Reference" "#PWR0113" (at 200.66 101.6 0)
       (effects (font (size 1.27 1.27)) hide)
     )
@@
     (instances
       (project "speedomobile"
-        (path "/33f5bcad-68ad-4ea6-9034-cdbd4086270c/f11e76c2-c975-435e-b3f1-8c0be3fa1a36"
-          (reference "#PWR?") (unit 1)
-        )
         (path "/33f5bcad-68ad-4ea6-9034-cdbd4086270c/51c364bc-8dcb-4f10-88b1-180da7ba62ce"
           (reference "#PWR0113") (unit 1)
@@
   (symbol (lib_id "Device:C") (at 213.36 101.6 0) (unit 1)
     (in_bom yes) (on_board yes) (dnp no) (fields_autoplaced)
-    (property "Reference" "C?" (at 217.17 100.33 0)
+    (property "Reference" "C18" (at 217.17 100.33 0)
       (effects (font (size 1.27 1.27)) (justify left))
     )
@@
     (instances
       (project "speedomobile"
-        (path "/33f5bcad-68ad-4ea6-9034-cdbd4086270c/f11e76c2-c975-435e-b3f1-8c0be3fa1a36"
-          (reference "C?") (unit 1)
-        )
         (path "/33f5bcad-68ad-4ea6-9034-cdbd4086270c/51c364bc-8dcb-4f10-88b1-180da7ba62ce"
           (reference "C18") (unit 1)
