File: speedomobile.kicad_sch (KiCad schematic)
At the start: 21 parts, among them J29 Conn_01x02, J30 Conn_01x06, J31 Conn_02x06_Odd_Even, J36 Conn_01x03, Q1 DMT6012LSS, SW1 SW_Push, U1 MCP1501-33xCH, U2 SC0918, U3 74AHCT367

Commit message: JLCJLCJLCJLC
Parts:
- removed J36: Conn_01x03, Connector_PinHeader_2.54mm:PinHeader_1x03_P2.54mm_Vertical, symbol Connector_Generic:Conn_01x03
Connections:
- no-connect marks 2 -> 3
Changed lines of the file:
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@@
   (junction (at 121.92 138.43) (diameter 0) (color 0 0 0 0)
   )
-  (junction (at 21.59 71.755) (diameter 0) (color 0 0 0 0)
-  )
   (junction (at 40.64 30.48) (diameter 0) (color 0 0 0 0)
   )
@@
   )
   (no_connect (at 134.62 151.13))
+  (no_connect (at 26.67 73.66))
   (no_connect (at 77.47 72.39))
   (wire (pts (xy 96.52 96.52) (xy 110.49 96.52))
@@
     (stroke (width 0) (type default))
   )
-  (wire (pts (xy 26.67 66.675) (xy 21.59 66.675))
-    (stroke (width 0) (type default))
-  )
   (wire (pts (xy 91.44 32.385) (xy 100.33 32.385))
     (stroke (width 0) (type default))
@@
     (stroke (width 0) (type default))
   )
-  (wire (pts (xy 21.59 71.755) (xy 21.59 72.39))
-    (stroke (width 0) (type default))
-  )
   (wire (pts (xy 135.89 86.36) (xy 151.13 86.36))
     (stroke (width 0) (type default))
@@
     (stroke (width 0) (type default))
   )
-  (wire (pts (xy 21.59 71.755) (xy 21.59 69.215))
-    (stroke (width 0) (type default))
-  )
   (wire (pts (xy 100.33 42.545) (xy 100.33 37.465))
     (stroke (width 0) (type default))
@@
   )
   (wire (pts (xy 109.22 173.99) (xy 121.92 173.99))
-    (stroke (width 0) (type default))
-  )
-  (wire (pts (xy 26.67 73.66) (xy 26.67 66.675))
     (stroke (width 0) (type default))
   )
@@
     )
   )
-  (symbol (lib_id "Connector_Generic:Conn_01x03") (at 16.51 69.215 180) (unit 1)
-    (in_bom yes) (on_board yes) (dnp no) (fields_autoplaced)
-    (property "Reference" "J36" (at 16.51 60.325 0)
-      (effects (font (size 1.27 1.27)))
-    )
-    (property "Value" "Conn_01x03" (at 16.51 62.865 0)
-      (effects (font (size 1.27 1.27)))
-    )
-    (property "Footprint" "Connector_PinHeader_2.54mm:PinHeader_1x03_P2.54mm_Vertical" (at 16.51 69.215 0)
-      (effects (font (size 1.27 1.27)) hide)
-    )
-    (property "Datasheet" "~" (at 16.51 69.215 0)
-      (effects (font (size 1.27 1.27)) hide)
-    )
-    (property "tme" "" (at 16.51 69.215 0)
-      (effects (font (size 1.27 1.27)) hide)
-    )
-    (pin "2")
-    (pin "3")
-    (pin "1")
-    (instances
-      (project "speedomobile"
-        (path "/33f5bcad-68ad-4ea6-9034-cdbd4086270c"
-          (reference "J36") (unit 1)
-        )
-      )
-    )
-  )
   (symbol (lib_id "power:GND") (at 190.5 156.21 0) (unit 1)
     (in_bom yes) (on_board yes) (dnp no) (fields_autoplaced)
@@
         )
       )
-    )
-  )
-  (symbol (lib_id "power:GND") (at 21.59 72.39 0) (unit 1)
-    (in_bom yes) (on_board yes) (dnp no) (fields_autoplaced)
-    (property "Reference" "#PWR0158" (at 21.59 78.74 0)
-      (effects (font (size 1.27 1.27)) hide)
-    )
-    (property "Value" "GND" (at 21.59 77.47 0)
-      (effects (font (size 1.27 1.27)))
-    )
-    (property "Footprint" "" (at 21.59 72.39 0)
-      (effects (font (size 1.27 1.27)) hide)
-    )
-    (property "Datasheet" "" (at 21.59 72.39 0)
-      (effects (font (size 1.27 1.27)) hide)
-    )
-    (pin "1")
-    (instances
-      (project "speedomobile"
-        (path "/33f5bcad-68ad-4ea6-9034-cdbd4086270c"
-          (reference "#PWR0158") (unit 1)
-        )
-      )

Commit message: 2 layers!
Connections:
- net GND: now also J31.2 (Pin_2); no longer J31.6 (Pin_6)
- net GPIO0: now also J31.3 (Pin_3); no longer J31.2 (Pin_2)
- net GPIO1: now also J31.4 (Pin_4); no longer J31.3 (Pin_3)
- net GPIO2: now also J31.5 (Pin_5); no longer J31.4 (Pin_4)
- net GPIO3: now also J31.6 (Pin_6); no longer J31.5 (Pin_5)
- net PWR1_PWM: no longer U2.27 (I2C0SCL/GP21)
- net PWR2_PWM: no longer U2.26 (I2C0SDA/GP20)
- no-connect marks 3 -> 5
Changed lines of the file:
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@@
   (junction (at 121.92 173.99) (diameter 0) (color 0 0 0 0)
   )
+  (no_connect (at 91.44 133.35))
   (no_connect (at 134.62 151.13))
+  (no_connect (at 91.44 130.81))
   (no_connect (at 26.67 73.66))
   (no_connect (at 77.47 72.39))
@@
     (stroke (width 0) (type default))
   )
+  (wire (pts (xy 113.03 29.845) (xy 121.92 29.845))
+    (stroke (width 0) (type default))
+  )
   (wire (pts (xy 77.47 85.09) (xy 91.44 85.09))
     (stroke (width 0) (type default))
@@
     (stroke (width 0) (type default))
   )
-  (wire (pts (xy 121.92 24.765) (xy 113.03 24.765))
+  (wire (pts (xy 125.095 24.765) (xy 113.03 24.765))
     (stroke (width 0) (type default))
   )
@@
     (stroke (width 0) (type default))
   )
-  (wire (pts (xy 113.03 29.845) (xy 125.095 29.845))
-    (stroke (width 0) (type default))
-  )
   (wire (pts (xy 91.44 29.845) (xy 100.33 29.845))
     (stroke (width 0) (type default))
@@
     (effects (font (size 1.27 1.27)) (justify left bottom))
   )
-  (label "PWR2_PWM" (at 91.44 130.81 180) (fields_autoplaced)
-    (effects (font (size 1.27 1.27)) (justify right bottom))
-  )
   (label "ADC" (at 203.2 82.55 0) (fields_autoplaced)
     (effects (font (size 1.27 1.27)) (justify left bottom))
@@
     (effects (font (size 1.27 1.27)) (justify left bottom))
   )
-  (label "GPIO3" (at 91.44 29.845 0) (fields_autoplaced)
-    (effects (font (size 1.27 1.27)) (justify left bottom))
+  (label "GPIO3" (at 121.92 29.845 180) (fields_autoplaced)
+    (effects (font (size 1.27 1.27)) (justify right bottom))
   )
   (label "UART" (at 52.07 176.53 0) (fields_autoplaced)
@@
     (effects (font (size 1.27 1.27)) (justify left bottom))
   )
-  (label "PWR1_PWM" (at 91.44 133.35 180) (fields_autoplaced)
-    (effects (font (size 1.27 1.27)) (justify right bottom))
-  )
   (label "GPIO4" (at 91.44 115.57 180) (fields_autoplaced)
     (effects (font (size 1.27 1.27)) (justify right bottom))
   )
-  (label "GPIO0" (at 121.92 24.765 180) (fields_autoplaced)
-    (effects (font (size 1.27 1.27)) (justify right bottom))
+  (label "GPIO0" (at 91.44 27.305 0) (fields_autoplaced)
+    (effects (font (size 1.27 1.27)) (justify left bottom))
   )
   (label "REMOTE_COMM" (at 91.44 135.89 180) (fields_autoplaced)
@@
     (effects (font (size 1.27 1.27)) (justify right bottom))
   )
-  (label "GPIO1" (at 91.44 27.305 0) (fields_autoplaced)
-    (effects (font (size 1.27 1.27)) (justify left bottom))
+  (label "GPIO1" (at 121.92 27.305 180) (fields_autoplaced)
+    (effects (font (size 1.27 1.27)) (justify right bottom))
   )
   (label "TSDZ2_TX" (at 91.44 100.33 180) (fields_autoplaced)
@@
     (effects (font (size 1.27 1.27)) (justify right bottom))
   )
-  (label "GPIO2" (at 121.92 27.305 180) (fields_autoplaced)
-    (effects (font (size 1.27 1.27)) (justify right bottom))
+  (label "GPIO2" (at 91.44 29.845 0) (fields_autoplaced)
+    (effects (font (size 1.27 1.27)) (justify left bottom))
   )
   (label "FAST_SCL" (at 96.52 101.6 0) (fields_autoplaced)
@@
         (path "/33f5bcad-68ad-4ea6-9034-cdbd4086270c"
           (reference "#PWR019") (unit 1)
+        )
+      )
+    )
+  )
+  (symbol (lib_id "power:GND") (at 125.095 24.765 0) (unit 1)
+    (in_bom yes) (on_board yes) (dnp no) (fields_autoplaced)
+    (property "Reference" "#PWR0152" (at 125.095 31.115 0)
+      (effects (font (size 1.27 1.27)) hide)
+    )
+    (property "Value" "GND" (at 125.095 29.21 0)
+      (effects (font (size 1.27 1.27)))
+    )
+    (property "Footprint" "" (at 125.095 24.765 0)
+      (effects (font (size 1.27 1.27)) hide)
+    )
+    (property "Datasheet" "" (at 125.095 24.765 0)
+      (effects (font (size 1.27 1.27)) hide)
+    )
+    (pin "1")
+    (instances
+      (project "speedomobile"
+        (path "/33f5bcad-68ad-4ea6-9034-cdbd4086270c"
+          (reference "#PWR0152") (unit 1)
         )
       )
@@
         )
       )
-    )
-  )
-  (symbol (lib_id "power:GND") (at 125.095 29.845 0) (unit 1)
-    (in_bom yes) (on_board yes) (dnp no) (fields_autoplaced)
-    (property "Reference" "#PWR0159" (at 125.095 36.195 0)
-      (effects (font (size 1.27 1.27)) hide)
-    )
-    (property "Value" "GND" (at 125.095 34.925 0)
-      (effects (font (size 1.27 1.27)))
-    )
-    (property "Footprint" "" (at 125.095 29.845 0)
-      (effects (font (size 1.27 1.27)) hide)
-    )
-    (property "Datasheet" "" (at 125.095 29.845 0)
-      (effects (font (size 1.27 1.27)) hide)
-    )
-    (pin "1")
-    (instances
-      (project "speedomobile"
-        (path "/33f5bcad-68ad-4ea6-9034-cdbd4086270c"
-          (reference "#PWR0159") (unit 1)
-        )
-      )

Commit message: Before flip
Parts:
- J31: mouser (none) -> 538-90130-1112
- R2: mouser (none) -> 791-WR12X4701FTL
- R3: mouser (none) -> 603-AC1206FR-101KL
- R4: value 190k -> 191k; mouser (none) -> 660-RK73H2BTTD1913F
Connections:
- net CS_SD: now also U2.2 (UART0RX/I2C0SCL/SPI0Cs/GP01); no longer U2.10 (I2C1SCL/SPI0TX/GP07)
- net GPIO0: now also U2.26 (I2C0SDA/GP20); no longer U2.16 (UART0TX/I2C0SDA/SPI1RX/GP12)
- net GPIO1: now also U2.27 (I2C0SCL/GP21); no longer U2.25 (I2C1SCL/SPI0TX/GP19)
- net GPIO2: now also U2.24 (I2C1SDA/SPI0CK/GP18); no longer U2.17 (UART0RX/I2C0SCL/SPI1Cs/GP13)
- net GPIO3: now also U2.25 (I2C1SCL/SPI0TX/GP19); no longer U2.24 (I2C1SDA/SPI0CK/GP18)
- net GPIO4: now also U2.22 (UART0RX/I2C0SCL/SPI0Cs/GP17); no longer U2.19 (I2C1SDA/SPI1CK/GP14)
- net GPIO5: now also U2.19 (I2C1SDA/SPI1CK/GP14); no longer U2.22 (UART0RX/I2C0SCL/SPI0Cs/GP17)
- net GPIO6: now also U2.21 (UART0TX/I2C0SDA/SPI0RX/GP16); no longer U2.20 (I2C1SCL/SPI1TX/GP15)
- net GPIO7: now also U2.20 (I2C1SCL/SPI1TX/GP15); no longer U2.21 (UART0TX/I2C0SDA/SPI0RX/GP16)
- net AUX_CK renamed AUX
- net AUX_TX: no longer names the net of U2.15 (I2C1SCL/SPI1TX/GP11)
- net AUX_TX: no longer J30.3 (Pin_3)
- net UART renamed UARTRX
- net UARTRX: now also U2.17 (UART0RX/I2C0SCL/SPI1Cs/GP13); no longer U2.2 (UART0RX/I2C0SCL/SPI0Cs/GP01)
- new net PPS: U2.10 (I2C1SCL/SPI0TX/GP07)
- new net UARTTX: J30.3 (Pin_3), U2.16 (UART0TX/I2C0SDA/SPI1RX/GP12)
- no-connect marks 5 -> 4
Other:
- sheet I2C devices ports: added PPS; removed none

Commit message: before expansion
Connections:
- net +3V3: now also J31.12 (Pin_12); no longer J31.11 (Pin_11)
- net +5VL: now also J31.11 (Pin_11); no longer J31.12 (Pin_12)
- net GND: now also U3.14 (I6); no longer U3.6 (I3)
- net HONK: now also U3.2 (I1); no longer U3.14 (I6)
- net HONK_5V: now also U3.3 (O1a); no longer U3.13 (O6b)
- net PPS: now also U2.9 (I2C1SDA/SPI0CK/GP06); no longer U2.10 (I2C1SCL/SPI0TX/GP07)
- net TSDZ2_BRAKE: now also U3.10 (I4); no longer U3.12 (I5)
- net TSDZ2_BRAKE_5V: now also U3.9 (O4a); no longer U3.11 (O5b)
- net TSDZ2_ON: now also U3.4 (I2); no longer U3.2 (I1)
- net TSDZ2_ON_5V: now also U3.5 (O2a); no longer U3.3 (O1a)
- net TSDZ2_TX: now also U3.6 (I3); no longer U3.10 (I4)
- net TSDZ2_TX_5V: now also U3.7 (O3a); no longer U3.9 (O4a)
- net VSPEED: now also U2.10 (I2C1SCL/SPI0TX/GP07), U3.12 (I5); no longer U2.9 (I2C1SDA/SPI0CK/GP06), U3.4 (I2)
- net VSPEED_5V: now also U3.11 (O5b); no longer U3.5 (O2a)
- net RESET: now reaches SW1.2, U2.30 (RUN)

Commit message: Prepare for merging
Parts:
- removed J30: Conn_01x06, Connector_JST:JST_XH_B6B-XH-A_1x06_P2.50mm_Vertical, symbol Connector_Generic:Conn_01x06
- added C5: 22u, Capacitor_SMD:C_1210_3225Metric, symbol Device:C
- added C6: 220u, Capacitor_THT:CP_Radial_D16.0mm_P7.50mm, symbol Device:C_Polarized
- added J11: JST_XH, Connector_JST:JST_XH_B4B-XH-A_1x04_P2.50mm_Vertical, symbol Connector_Generic:Conn_01x04
Connections:
- net AUX is gone; now on net TSDZ2_TX: U2.14 (I2C1SDA/SPI1CK/GP10)
- net +5VL: now also C5.1, C6.1, J11.1 (Pin_1)
- net GND: now also C5.2, C6.2, J11.4 (Pin_4)
- net HONK: now also U3.10 (I4); no longer U3.2 (I1)
- net HONK_5V: now also U3.9 (O4a); no longer U3.3 (O1a)
- net TSDZ2_BRAKE: now also U3.12 (I5); no longer U3.10 (I4)
- net TSDZ2_BRAKE_5V: now also U3.11 (O5b); no longer U3.9 (O4a)
- net TSDZ2_ON: now also U3.6 (I3); no longer U3.4 (I2)
- net TSDZ2_ON_5V: now also U3.7 (O3a); no longer U3.5 (O2a)
- net TSDZ2_RX: now also U2.15 (I2C1SCL/SPI1TX/GP11); no longer U2.12 (UART1RX/I2C0SCL/SPI1Cs/GP09)
- net TSDZ2_TX: now also U3.2 (I1); no longer U2.11 (UART1TX/I2C0SDA/SPI1RX/GP08), U3.6 (I3)
- net TSDZ2_TX_5V: now also U3.3 (O1a); no longer U3.7 (O3a)
- net UARTRX: now also J11.3 (Pin_3)
- net UARTTX: now also J11.2 (Pin_2)
- net VSPEED: now also U3.4 (I2); no longer U3.12 (I5)
- net VSPEED_5V: now also U3.5 (O2a); no longer U3.11 (O5b)
- net HONK_48V: now reaches J29.2 (Pin_2), Q1.5 (D), Q1.6 (D), Q1.7 (D), Q1.8 (D)
- net VREF renamed +3.3VA
- new net GPS_RX: U2.12 (UART1RX/I2C0SCL/SPI1Cs/GP09)
- new net GPS_TX: U2.11 (UART1TX/I2C0SDA/SPI1RX/GP08)
- no-connect marks 4 -> 3
Other:
- removed sheet power
- added sheet GPS (GPS.kicad_sch)
- sheet Analog input ports: added none; removed I5V, Imotor
- sheet I2C devices ports: added RESET_M9N; removed none
- moved on the sheet: J29
