File: hardware/i2c-daughter-board/i2c-daughter-board.kicad_sch (KiCad schematic)
At the start: 38 parts, among them J1 Conn_01x05, SW1 PEC11H, SW2 PEC11H, U13 TCA9617A, U5 PCF8574

Commit message: Updating images & 3d models
Parts:
- U1: footprint breakboard:PN532 -> additional:PN532
- U2: footprint breakboard:HD44780_PCF8574T -> additional:HD44780_PCF8574T
