File: hardware/i2c-daughter-board-measurement/i2c-daughter-board-measurement.kicad_sch (KiCad schematic)
At the start: 12 parts, among them J1 Conn_01x04, U5 PCF8574

Commit message: Updating images & 3d models
Parts:
- U3: footprint breakboard:bme680 -> additional:bme680
Changed lines of the file:
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@@
     (pin "1")
     (instances
-      (project "speedomobile-i2cmeasurement"
+      (project "i2c-daughter-board-measurement"
         (path "/e3e71c85-246e-4ad0-9afc-06ca0922ac40"
           (reference "H1") (unit 1)
@@
     (pin "1")
     (instances
-      (project "speedomobile-i2cmeasurement"
+      (project "i2c-daughter-board-measurement"
         (path "/e3e71c85-246e-4ad0-9afc-06ca0922ac40"
           (reference "#FLG02") (unit 1)
@@
         )
       )
-      (project "speedomobile-i2cmeasurement"
+      (project "i2c-daughter-board-measurement"
         (path "/e3e71c85-246e-4ad0-9afc-06ca0922ac40"
           (reference "#PWR043") (unit 1)
@@
     (pin "1")
     (instances
-      (project "speedomobile-i2cmeasurement"
+      (project "i2c-daughter-board-measurement"
         (path "/e3e71c85-246e-4ad0-9afc-06ca0922ac40"
           (reference "#PWR06") (unit 1)
@@
         )
       )
-      (project "speedomobile-i2cmeasurement"
+      (project "i2c-daughter-board-measurement"
         (path "/e3e71c85-246e-4ad0-9afc-06ca0922ac40"
           (reference "#PWR044") (unit 1)
@@
     (pin "1")
     (instances
-      (project "speedomobile-i2cmeasurement"
+      (project "i2c-daughter-board-measurement"
         (path "/e3e71c85-246e-4ad0-9afc-06ca0922ac40"
           (reference "H2") (unit 1)
@@
     (pin "1")
     (instances
-      (project "speedomobile-i2cmeasurement"
+      (project "i2c-daughter-board-measurement"
         (path "/e3e71c85-246e-4ad0-9afc-06ca0922ac40"
           (reference "#PWR013") (unit 1)
@@
     (pin "1")
     (instances
-      (project "speedomobile-i2cmeasurement"
+      (project "i2c-daughter-board-measurement"
         (path "/e3e71c85-246e-4ad0-9afc-06ca0922ac40"
           (reference "#PWR03") (unit 1)
@@
     (pin "1")
     (instances
-      (project "speedomobile-i2cmeasurement"
+      (project "i2c-daughter-board-measurement"
         (path "/e3e71c85-246e-4ad0-9afc-06ca0922ac40"
           (reference "#FLG03") (unit 1)
@@
     (pin "1")
     (instances
-      (project "speedomobile-i2cmeasurement"
+      (project "i2c-daughter-board-measurement"
         (path "/e3e71c85-246e-4ad0-9afc-06ca0922ac40"
           (reference "#PWR02") (unit 1)
@@
     (pin "1")
     (instances
-      (project "speedomobile-i2cmeasurement"
+      (project "i2c-daughter-board-measurement"
         (path "/e3e71c85-246e-4ad0-9afc-06ca0922ac40"
           (reference "#PWR016") (unit 1)
@@
       (effects (font (size 1.27 1.27)))
     )
-    (property "Footprint" "breakboard:bme680" (at 50.165 104.14 0)
+    (property "Footprint" "additional:bme680" (at 50.165 104.14 0)
       (effects (font (size 1.27 1.27)) hide)
     )
@@
     (pin "7")
     (instances
-      (project "speedomobile-i2cmeasurement"
+      (project "i2c-daughter-board-measurement"
         (path "/e3e71c85-246e-4ad0-9afc-06ca0922ac40"
           (reference "U3") (unit 1)
@@
     (pin "1")
     (instances
-      (project "speedomobile-i2cmeasurement"
+      (project "i2c-daughter-board-measurement"
         (path "/e3e71c85-246e-4ad0-9afc-06ca0922ac40"
           (reference "#PWR047") (unit 1)
@@
         )
       )
-      (project "speedomobile-i2cmeasurement"
+      (project "i2c-daughter-board-measurement"
         (path "/e3e71c85-246e-4ad0-9afc-06ca0922ac40"
           (reference "C5") (unit 1)
@@
         )
       )
-      (project "speedomobile-i2cmeasurement"
+      (project "i2c-daughter-board-measurement"
         (path "/e3e71c85-246e-4ad0-9afc-06ca0922ac40"
           (reference "#PWR025") (unit 1)
@@
         )
       )
-      (project "speedomobile-i2cmeasurement"
+      (project "i2c-daughter-board-measurement"
         (path "/e3e71c85-246e-4ad0-9afc-06ca0922ac40"
           (reference "#PWR04") (unit 1)
@@
         )
       )
-      (project "speedomobile-i2cmeasurement"
+      (project "i2c-daughter-board-measurement"
         (path "/e3e71c85-246e-4ad0-9afc-06ca0922ac40"
           (reference "#PWR026") (unit 1)
@@
         )
       )
-      (project "speedomobile-i2cmeasurement"
+      (project "i2c-daughter-board-measurement"
         (path "/e3e71c85-246e-4ad0-9afc-06ca0922ac40"
           (reference "C6") (unit 1)
@@
     (pin "11")
     (instances
-      (project "speedomobile-i2cmeasurement"
+      (project "i2c-daughter-board-measurement"
         (path "/e3e71c85-246e-4ad0-9afc-06ca0922ac40"
           (reference "U5") (unit 1)
@@
     (pin "1")
     (instances
-      (project "speedomobile-i2cmeasurement"
+      (project "i2c-daughter-board-measurement"
         (path "/e3e71c85-246e-4ad0-9afc-06ca0922ac40"
           (reference "#PWR010") (unit 1)
@@
     (pin "1")
     (instances
-      (project "speedomobile-i2cmeasurement"
+      (project "i2c-daughter-board-measurement"
         (path "/e3e71c85-246e-4ad0-9afc-06ca0922ac40"
           (reference "#PWR012") (unit 1)
@@
     (pin "1")
     (instances
-      (project "speedomobile-i2cmeasurement"
+      (project "i2c-daughter-board-measurement"
         (path "/e3e71c85-246e-4ad0-9afc-06ca0922ac40"
           (reference "#PWR015") (unit 1)
@@
     (pin "1")
     (instances
-      (project "speedomobile-i2cmeasurement"
+      (project "i2c-daughter-board-measurement"
         (path "/e3e71c85-246e-4ad0-9afc-06ca0922ac40"
           (reference "H3") (unit 1)
@@
         )
       )
-      (project "speedomobile-i2cmeasurement"
+      (project "i2c-daughter-board-measurement"
         (path "/e3e71c85-246e-4ad0-9afc-06ca0922ac40"
           (reference "#PWR045") (unit 1)
@@
         )
       )
-      (project "speedomobile-i2cmeasurement"
+      (project "i2c-daughter-board-measurement"
         (path "/e3e71c85-246e-4ad0-9afc-06ca0922ac40"
           (reference "#PWR028") (unit 1)
@@
     (pin "1")
     (instances
-      (project "speedomobile-i2cmeasurement"
+      (project "i2c-daughter-board-measurement"
         (path "/e3e71c85-246e-4ad0-9afc-06ca0922ac40"
           (reference "#PWR014") (unit 1)
@@
         )
       )
-      (project "speedomobile-i2cmeasurement"
+      (project "i2c-daughter-board-measurement"
         (path "/e3e71c85-246e-4ad0-9afc-06ca0922ac40"
           (reference "C14") (unit 1)
@@
     (pin "1")
     (instances
-      (project "speedomobile-i2cmeasurement"
+      (project "i2c-daughter-board-measurement"
         (path "/e3e71c85-246e-4ad0-9afc-06ca0922ac40"
           (reference "H4") (unit 1)
@@
     (pin "1")
     (instances
-      (project "speedomobile-i2cmeasurement"
+      (project "i2c-daughter-board-measurement"
         (path "/e3e71c85-246e-4ad0-9afc-06ca0922ac40"
           (reference "#PWR01") (unit 1)
@@
     (pin "1")
     (instances
-      (project "speedomobile-i2cmeasurement"
+      (project "i2c-daughter-board-measurement"
         (path "/e3e71c85-246e-4ad0-9afc-06ca0922ac40"
           (reference "#PWR041") (unit 1)
@@
     (pin "1")
     (instances
-      (project "speedomobile-i2cmeasurement"
+      (project "i2c-daughter-board-measurement"
         (path "/e3e71c85-246e-4ad0-9afc-06ca0922ac40"
           (reference "#PWR05") (unit 1)
@@
     (pin "2")
     (instances
-      (project "speedomobile-i2cmeasurement"
+      (project "i2c-daughter-board-measurement"
         (path "/e3e71c85-246e-4ad0-9afc-06ca0922ac40"
           (reference "J1") (unit 1)
@@
         )
       )
-      (project "speedomobile-i2cmeasurement"
+      (project "i2c-daughter-board-measurement"
         (path "/e3e71c85-246e-4ad0-9afc-06ca0922ac40"
           (reference "SYMB1") (unit 1)
@@
     (pin "6")
     (instances
-      (project "speedomobile-i2cmeasurement"
+      (project "i2c-daughter-board-measurement"
         (path "/e3e71c85-246e-4ad0-9afc-06ca0922ac40"
           (reference "U1") (unit 1)
